Commit message: Aruco detection Transform (TF) code V1

File: ws/src/pfe/description/my_robot.urdf.xacro (robot description, xacro)
@@ -3,9 +3,10 @@
     <xacro:include filename="include_tags.urdf.xacro" />
     <link name="world"></link>
-    <joint name="base_joint" type="planar">
+    <joint name="base_joint" type="prismatic">
         <origin xyz="1.5 1.0 0.0617" rpy="0 0 0" />
         <parent link="world" />
         <child link="base_link" />
-        <axis xyz="0 0 1" />
+        <axis xyz="0.7071 0.7071 0"/>
+        <limit lower="0.0" upper="1.0" effort="1000" velocity="0.5"/>
     </joint>
     <link name="base_link">
@@ -30,5 +31,5 @@
     </link>
     <joint name="arducam_joint" type="fixed">
-        <origin xyz="0 0 .626" rpy="{-pi/12} 0 0" />
+        <origin xyz="0 0 .626" rpy="-0.261799 0 0" />
         <parent link="base_link" />
         <child link="arducam_link" />
@@ -53,4 +54,5 @@
             <origin xyz="0 0 .0025" rpy="0 0 0" />
         </xacro:inertial_box>
-    <xacro:include filename="example_gazebo.xacro" />
+    </link>
+    <!-- <xacro:include filename="example_gazebo.xacro" /> -->
 </robot>

Commit message: Added ArucoNavGoal for camera goal pose

File: ws/src/pfe/description/my_robot.urdf.xacro (robot description, xacro)
@@ -1,58 +1,257 @@
 <?xml version="1.0"?>
-<robot xmlns:xacro="http://www.ros.org/wiki/xacro"  name="robot" >
-    <xacro:include filename="include_tags.urdf.xacro" />
-    <link name="world"></link>
-    <joint name="base_joint" type="prismatic">
-        <origin xyz="1.5 1.0 0.0617" rpy="0 0 0" />
-        <parent link="world" />
-        <child link="base_link" />
-        <axis xyz="0.7071 0.7071 0"/>
-        <limit lower="0.0" upper="1.0" effort="1000" velocity="0.5"/>
-    </joint>
-    <link name="base_link">
-        <visual>
-            <origin xyz="0 0 .0025" rpy="0 0 0" />
-            <geometry>
-                <box size=".22 .24 .005" />
-            </geometry>
-            <material name="green">
-                <color rgba="0.2 1 0.2 1"/>
-            </material>
-        </visual>
-        <collision>
-            <origin xyz="0 0 .0025" rpy="0 0 0" />
-            <geometry>
-                <box size=".22 .24 .005" />
-            </geometry>
-        </collision>
-        <xacro:inertial_box mass="2.0" x=".22" y=".24" z=".005">
-            <origin xyz="0 0 .0025" rpy="0 0 0" />
-        </xacro:inertial_box>
-    </link>
-    <joint name="arducam_joint" type="fixed">
-        <origin xyz="0 0 .626" rpy="-0.261799 0 0" />
-        <parent link="base_link" />
-        <child link="arducam_link" />
-    </joint>
-    <link name="arducam_link">
-        <visual>
-            <origin xyz="0 0 .0025" rpy="0 0 0" />
-            <geometry>
-                <box size=".02 .02 .02" />
-            </geometry>
-            <material name="black">
-                <color rgba="0 0 0 1"/>
-            </material>
-        </visual>
-        <collision>
-            <origin xyz="0 0 .0025" rpy="0 0 0" />
-            <geometry>
-                <box size=".02 .02 .02" />
-            </geometry>
-        </collision>
-        <xacro:inertial_box mass="0.1" x="0.02" y="0.02" z=".02">
-            <origin xyz="0 0 .0025" rpy="0 0 0" />
-        </xacro:inertial_box>
-    </link>
-    <!-- <xacro:include filename="example_gazebo.xacro" /> -->
+<robot name="pfe_robot">
+  <!-- ===================== WORLD LINK ===================== -->
+  <link name="world"/>
+  <!-- ===================== BASE LINK ===================== -->
+  <link name="Base-v1">
+    <visual>
+      <origin xyz="0 0 0" rpy="0 0 0"/>
+      <geometry>
+        <!-- <mesh filename="package://pfe/meshes/Base-v1.stl" scale="0.001 0.001 0.001"/>-->
+      </geometry>
+    </visual>
+    <collision>
+      <origin xyz="0 0 0" rpy="0 0 0"/>
+      <geometry>
+        <mesh filename="package://pfe/meshes/Base-v1.stl" scale="0.001 0.001 0.001"/>
+      </geometry>
+    </collision>
+    <inertial>
+      <origin xyz="0 0 0" rpy="0 0 0"/>
+      <mass value="2.0"/>
+      <inertia ixx="0.01" ixy="0" ixz="0" iyy="0.01" iyz="0" izz="0.01"/>
+    </inertial>
+  </link>
+  <joint name="world_to_base" type="fixed">
+    <parent link="world"/>
+    <child link="Base-v1"/>
+    <origin xyz="0 0 0" rpy="0 0 0"/>
+  </joint>
+  <!-- ===================== MOUNT TO WHEEL LINKS ===================== -->
+  <link name="MountToWheel-v1_a">
+    <visual>
+      <origin xyz="0 0 0" rpy="0 0 0"/>
+      <geometry>
+        <mesh filename="package://pfe/meshes/MountToWheel-v1.stl" scale="0.001 0.001 0.001"/>
+      </geometry>
+    </visual>
+    <collision>
+      <origin xyz="0 0 0" rpy="0 0 0"/>
+      <geometry>
+        <mesh filename="package://pfe/meshes/MountToWheel-v1.stl" scale="0.001 0.001 0.001"/>
+      </geometry>
+    </collision>
+    <inertial>
+      <origin xyz="0 0 0" rpy="0 0 0"/>
+      <mass value="0.1"/>
+      <inertia ixx="0.0001" ixy="0" ixz="0" iyy="0.0001" iyz="0" izz="0.0001"/>
+    </inertial>
+  </link>
+  <link name="MountToWheel-v1_b">
+    <visual>
+      <origin xyz="0 0 0" rpy="0 0 0"/>
+      <geometry>
+        <mesh filename="package://pfe/meshes/MountToWheel-v1.stl" scale="0.001 0.001 0.001"/>
+      </geometry>
+    </visual>
+    <collision>
+      <origin xyz="0 0 0" rpy="0 0 0"/>
+      <geometry>
+        <mesh filename="package://pfe/meshes/MountToWheel-v1.stl" scale="0.001 0.001 0.001"/>
+      </geometry>
+    </collision>
+    <inertial>
+      <origin xyz="0 0 0" rpy="0 0 0"/>
+      <mass value="0.1"/>
+      <inertia ixx="0.0001" ixy="0" ixz="0" iyy="0.0001" iyz="0" izz="0.0001"/>
+    </inertial>
+  </link>
+  <link name="MountToWheel-v1_c">
+    <visual>
+      <origin xyz="0 0 0" rpy="0 0 0"/>
+      <geometry>
+        <mesh filename="package://pfe/meshes/MountToWheel-v1.stl" scale="0.001 0.001 0.001"/>
+      </geometry>
+    </visual>
+    <collision>
+      <origin xyz="0 0 0" rpy="0 0 0"/>
+      <geometry>
+        <mesh filename="package://pfe/meshes/MountToWheel-v1.stl" scale="0.001 0.001 0.001"/>
+      </geometry>
+    </collision>
+    <inertial>
+      <origin xyz="0 0 0" rpy="0 0 0"/>
+      <mass value="0.1"/>
+      <inertia ixx="0.0001" ixy="0" ixz="0" iyy="0.0001" iyz="0" izz="0.0001"/>
+    </inertial>
+  </link>
+  <link name="MountToWheel-v1_d">
+    <visual>
+      <origin xyz="0 0 0" rpy="0 0 0"/>
+      <geometry>
+        <mesh filename="package://pfe/meshes/MountToWheel-v1.stl" scale="0.001 0.001 0.001"/>
+      </geometry>
+    </visual>
+    <collision>
+      <origin xyz="0 0 0" rpy="0 0 0"/>
+      <geometry>
+        <mesh filename="package://pfe/meshes/MountToWheel-v1.stl" scale="0.001 0.001 0.001"/>
+      </geometry>
+    </collision>
+    <inertial>
+      <origin xyz="0 0 0" rpy="0 0 0"/>
+      <mass value="0.1"/>
+      <inertia ixx="0.0001" ixy="0" ixz="0" iyy="0.0001" iyz="0" izz="0.0001"/>
+    </inertial>
+  </link>
+  <!-- ===================== WHEEL JOINT LINKS ===================== -->
+  <link name="WheelJoint-v1_a">
+    <visual>
+      <origin xyz="0 0 0" rpy="0 0 0"/>
+      <geometry>
+        <mesh filename="package://pfe/meshes/WheelJoint-v1.stl" scale="0.001 0.001 0.001"/>
+      </geometry>
+    </visual>
+    <collision>
+      <origin xyz="0 0 0" rpy="0 0 0"/>
+      <geometry>
+        <mesh filename="package://pfe/meshes/WheelJoint-v1.stl" scale="0.001 0.001 0.001"/>
+      </geometry>
+    </collision>
+    <inertial>
+      <origin xyz="0 0 0" rpy="0 0 0"/>
+      <mass value="0.05"/>
+      <inertia ixx="0.00005" ixy="0" ixz="0" iyy="0.00005" iyz="0" izz="0.00005"/>
+    </inertial>
+  </link>
+  <link name="WheelJoint-v1_b">
+    <visual>
+      <origin xyz="0 0 0" rpy="0 0 0"/>
+      <geometry>
+        <mesh filename="package://pfe/meshes/WheelJoint-v1.stl" scale="0.001 0.001 0.001"/>
+      </geometry>
+    </visual>
+    <collision>
+      <origin xyz="0 0 0" rpy="0 0 0"/>
+      <geometry>
+        <mesh filename="package://pfe/meshes/WheelJoint-v1.stl" scale="0.001 0.001 0.001"/>
+      </geometry>
+    </collision>
+    <inertial>
+      <origin xyz="0 0 0" rpy="0 0 0"/>
+      <mass value="0.05"/>
+      <inertia ixx="0.00005" ixy="0" ixz="0" iyy="0.00005" iyz="0" izz="0.00005"/>
+    </inertial>
+  </link>
+  <link name="WheelJoint-v1_c">
+    <visual>
+      <origin xyz="0 0 0" rpy="0 0 0"/>
+      <geometry>
+        <mesh filename="package://pfe/meshes/WheelJoint-v1.stl" scale="0.001 0.001 0.001"/>
+      </geometry>
+    </visual>
+    <collision>
+      <origin xyz="0 0 0" rpy="0 0 0"/>
+      <geometry>
+        <mesh filename="package://pfe/meshes/WheelJoint-v1.stl" scale="0.001 0.001 0.001"/>
+      </geometry>
+    </collision>
+    <inertial>
+      <origin xyz="0 0 0" rpy="0 0 0"/>
+      <mass value="0.05"/>
+      <inertia ixx="0.00005" ixy="0" ixz="0" iyy="0.00005" iyz="0" izz="0.00005"/>
+    </inertial>
+  </link>
+  <link name="WheelJoint-v1_d">
+    <visual>
+      <origin xyz="0 0 0" rpy="0 0 0"/>
+      <geometry>
+        <mesh filename="package://pfe/meshes/WheelJoint-v1.stl" scale="0.001 0.001 0.001"/>
+      </geometry>
+    </visual>
+    <collision>
+      <origin xyz="0 0 0" rpy="0 0 0"/>
+      <geometry>
+        <mesh filename="package://pfe/meshes/WheelJoint-v1.stl" scale="0.001 0.001 0.001"/>
+      </geometry>
+    </collision>
+    <inertial>
+      <origin xyz="0 0 0" rpy="0 0 0"/>
+      <mass value="0.05"/>
+      <inertia ixx="0.00005" ixy="0" ixz="0" iyy="0.00005" iyz="0" izz="0.00005"/>
+    </inertial>
+  </link>
+  <!-- ===================== ARDUCAM LINK ===================== -->
+  <link name="arducam_link">
+    <visual>
+      <origin xyz="0 0 0" rpy="0 0 0"/>
+      <geometry>
+        <mesh filename="package://pfe/meshes/arducam_link-v1.stl" scale="0.001 0.001 0.001"/>
+      </geometry>
+    </visual>
+    <collision>
+      <origin xyz="0 0 0" rpy="0 0 0"/>
+      <geometry>
+        <mesh filename="package://pfe/meshes/arducam_link-v1.stl" scale="0.001 0.001 0.001"/>
+      </geometry>
+    </collision>
+    <inertial>
+      <origin xyz="0 0 0" rpy="0 0 0"/>
+      <mass value="0.1"/>
+      <inertia ixx="0.0001" ixy="0" ixz="0" iyy="0.0001" iyz="0" izz="0.0001"/>
+    </inertial>
+  </link>
+  <!-- ===================== JOINTS ===================== -->
+  <!-- Base to MountToWheel -->
+  <joint name="Base_to_MountToWheel_a" type="fixed">
+    <parent link="Base-v1"/>
+    <child link="MountToWheel-v1_a"/>
+    <origin xyz="0.163 0.215 0.005" rpy="3.1416 0 3.1416"/>
+  </joint>
+  <joint name="Base_to_MountToWheel_b" type="fixed">
+    <parent link="Base-v1"/>
+    <child link="MountToWheel-v1_b"/>
+    <origin xyz="0.035 0.215 0.005" rpy="0 0 3.1416"/>
+  </joint>
+  <joint name="Base_to_MountToWheel_c" type="fixed">
+    <parent link="Base-v1"/>
+    <child link="MountToWheel-v1_c"/>
+    <origin xyz="0.077 0.005 0.005" rpy="0 0 3.1416"/>
+  </joint>
+  <joint name="Base_to_MountToWheel_d" type="fixed">
+    <parent link="Base-v1"/>
+    <child link="MountToWheel-v1_d"/>
+    <origin xyz="0.205 0.005 0.005" rpy="3.1416 0 3.1416"/>
+  </joint>
+  <!-- MountToWheel to WheelJoint -->
+  <joint name="MountToWheel_a_to_WheelJoint_a" type="continuous">
+    <parent link="MountToWheel-v1_a"/>
+    <child link="WheelJoint-v1_a"/>
+    <origin xyz="0.021 0.0192 0.027" rpy="-1.5708 0 0"/>
+    <axis xyz="0 0 1"/>
+  </joint>
+  <joint name="MountToWheel_b_to_WheelJoint_b" type="continuous">
+    <parent link="MountToWheel-v1_b"/>
+    <child link="WheelJoint-v1_b"/>
+    <origin xyz="0.021 -0.0192 -0.027" rpy="1.5708 0 0"/>
+    <axis xyz="0 0 1"/>
+  </joint>
+  <joint name="MountToWheel_c_to_WheelJoint_c" type="continuous">
+    <parent link="MountToWheel-v1_c"/>
+    <child link="WheelJoint-v1_c"/>
+    <origin xyz="-0.021 0.0192 -0.027" rpy="1.5708 0 0"/>
+    <axis xyz="0 0 -1"/>
+  </joint>
+  <joint name="MountToWheel_d_to_WheelJoint_d" type="continuous">
+    <parent link="MountToWheel-v1_d"/>
+    <child link="WheelJoint-v1_d"/>
+    <origin xyz="-0.021 -0.0192 0.027" rpy="-1.5708 0 0"/>
+    <axis xyz="0 0 -1"/>
+  </joint>
+  <!-- Base to Arducam -->
+  <joint name="Base_to_arducam" type="fixed">
+    <parent link="Base-v1"/>
+    <child link="arducam_link"/>
+    <origin xyz="0 0 0.626" rpy="-0.2618 0 0"/>
+  </joint>
 </robot>

Commit message: Changes for URDF

File: ws/src/pfe/description/my_robot.urdf.xacro (robot description, xacro)
@@ -2,7 +2,7 @@
 <robot name="pfe_robot">
   <!-- ===================== WORLD LINK ===================== -->
-  <link name="world"/>
+  <link name="map"/>
   <!-- ===================== BASE LINK ===================== -->
-  <link name="Base-v1">
+  <link name="base_link">
     <visual>
       <origin xyz="0 0 0" rpy="0 0 0"/>
@@ -23,7 +23,7 @@
     </inertial>
   </link>
-  <joint name="world_to_base" type="fixed">
-    <parent link="world"/>
-    <child link="Base-v1"/>
+  <joint name="map_to_base" type="fixed">
+    <parent link="map"/>
+    <child link="base_link"/>
     <origin xyz="0 0 0" rpy="0 0 0"/>
   </joint>
@@ -204,21 +204,21 @@
   <!-- ===================== JOINTS ===================== -->
   <!-- Base to MountToWheel -->
-  <joint name="Base_to_MountToWheel_a" type="fixed">
-    <parent link="Base-v1"/>
+  <joint name="base_to_MountToWheel_a" type="fixed">
+    <parent link="base_link"/>
     <child link="MountToWheel-v1_a"/>
     <origin xyz="0.163 0.215 0.005" rpy="3.1416 0 3.1416"/>
   </joint>
-  <joint name="Base_to_MountToWheel_b" type="fixed">
-    <parent link="Base-v1"/>
+  <joint name="base_to_MountToWheel_b" type="fixed">
+    <parent link="base_link"/>
     <child link="MountToWheel-v1_b"/>
     <origin xyz="0.035 0.215 0.005" rpy="0 0 3.1416"/>
   </joint>
-  <joint name="Base_to_MountToWheel_c" type="fixed">
-    <parent link="Base-v1"/>
+  <joint name="base_to_MountToWheel_c" type="fixed">
+    <parent link="base_link"/>
     <child link="MountToWheel-v1_c"/>
     <origin xyz="0.077 0.005 0.005" rpy="0 0 3.1416"/>
   </joint>
-  <joint name="Base_to_MountToWheel_d" type="fixed">
-    <parent link="Base-v1"/>
+  <joint name="base_to_MountToWheel_d" type="fixed">
+    <parent link="base_link"/>
     <child link="MountToWheel-v1_d"/>
     <origin xyz="0.205 0.005 0.005" rpy="3.1416 0 3.1416"/>
@@ -250,6 +250,6 @@
   </joint>
   <!-- Base to Arducam -->
-  <joint name="Base_to_arducam" type="fixed">
-    <parent link="Base-v1"/>
+  <joint name="base_to_arducam" type="fixed">
+    <parent link="base_link"/>
     <child link="arducam_link"/>
     <origin xyz="0 0 0.626" rpy="-0.2618 0 0"/>
