Commit message: URDF changes to include manip

File: ws/src/pfe/description/my_robot.urdf.xacro (robot description, xacro)
@@ -1,26 +1,8 @@
 <?xml version="1.0"?>
 <robot name="pfe_robot">
-  <!-- ===================== WORLD LINK ===================== -->
+  <!-- ===================== WORLD ===================== -->
   <link name="map"/>
-  <!-- ===================== BASE LINK ===================== -->
-  <link name="base_link">
-    <visual>
-      <origin xyz="0 0 0" rpy="0 0 0"/>
-      <geometry>
-        <!-- <mesh filename="package://pfe/meshes/Base-v1.stl" scale="0.001 0.001 0.001"/>-->
-      </geometry>
-    </visual>
-    <collision>
-      <origin xyz="0 0 0" rpy="0 0 0"/>
-      <geometry>
-        <mesh filename="package://pfe/meshes/Base-v1.stl" scale="0.001 0.001 0.001"/>
-      </geometry>
-    </collision>
-    <inertial>
-      <origin xyz="0 0 0" rpy="0 0 0"/>
-      <mass value="2.0"/>
-      <inertia ixx="0.01" ixy="0" ixz="0" iyy="0.01" iyz="0" izz="0.01"/>
-    </inertial>
-  </link>
+  <!-- ===================== ROS BASE ===================== -->
+  <link name="base_link"/>
   <joint name="map_to_base" type="fixed">
     <parent link="map"/>
@@ -28,10 +10,17 @@
     <origin xyz="0 0 0" rpy="0 0 0"/>
   </joint>
-  <!-- ===================== MOUNT TO WHEEL LINKS ===================== -->
-  <link name="MountToWheel-v1_a">
+  <!-- ===================== CAD WRAPPER (Fusion frame) ===================== -->
+  <!-- Fusion: +x backward, +y right  => rotate CAD frame by pi about Z to match ROS -->
+  <link name="base_cad">
+    <inertial>
+      <origin xyz="-0.181130474842482 0.10958995900517023 -0.10051074270429218" rpy="0 0 0"/>
+      <mass value="10.802255131301344"/>
+      <inertia ixx="0.11142549471720897" iyy="0.15234586542751433" izz="0.15214678916514196"
+               ixy="0.0002653832816470656" iyz="0.00027410838368888666" ixz="0.009773387741291757"/>
+    </inertial>
     <visual>
       <origin xyz="0 0 0" rpy="0 0 0"/>
       <geometry>
-        <mesh filename="package://pfe/meshes/MountToWheel-v1.stl" scale="0.001 0.001 0.001"/>
+        <mesh filename="package://pfe/meshes/base_link-v3.stl" scale="0.001 0.001 0.001"/>
       </geometry>
     </visual>
@@ -39,219 +28,207 @@
       <origin xyz="0 0 0" rpy="0 0 0"/>
       <geometry>
-        <mesh filename="package://pfe/meshes/MountToWheel-v1.stl" scale="0.001 0.001 0.001"/>
-      </geometry>
-    </collision>
-    <inertial>
-      <origin xyz="0 0 0" rpy="0 0 0"/>
-      <mass value="0.1"/>
-      <inertia ixx="0.0001" ixy="0" ixz="0" iyy="0.0001" iyz="0" izz="0.0001"/>
-    </inertial>
-  </link>
-  <link name="MountToWheel-v1_b">
-    <visual>
-      <origin xyz="0 0 0" rpy="0 0 0"/>
-      <geometry>
-        <mesh filename="package://pfe/meshes/MountToWheel-v1.stl" scale="0.001 0.001 0.001"/>
-      </geometry>
-    </visual>
-    <collision>
-      <origin xyz="0 0 0" rpy="0 0 0"/>
-      <geometry>
-        <mesh filename="package://pfe/meshes/MountToWheel-v1.stl" scale="0.001 0.001 0.001"/>
-      </geometry>
-    </collision>
-    <inertial>
-      <origin xyz="0 0 0" rpy="0 0 0"/>
-      <mass value="0.1"/>
-      <inertia ixx="0.0001" ixy="0" ixz="0" iyy="0.0001" iyz="0" izz="0.0001"/>
-    </inertial>
-  </link>
-  <link name="MountToWheel-v1_c">
-    <visual>
-      <origin xyz="0 0 0" rpy="0 0 0"/>
-      <geometry>
-        <mesh filename="package://pfe/meshes/MountToWheel-v1.stl" scale="0.001 0.001 0.001"/>
-      </geometry>
-    </visual>
-    <collision>
-      <origin xyz="0 0 0" rpy="0 0 0"/>
-      <geometry>
-        <mesh filename="package://pfe/meshes/MountToWheel-v1.stl" scale="0.001 0.001 0.001"/>
-      </geometry>
-    </collision>
-    <inertial>
-      <origin xyz="0 0 0" rpy="0 0 0"/>
-      <mass value="0.1"/>
-      <inertia ixx="0.0001" ixy="0" ixz="0" iyy="0.0001" iyz="0" izz="0.0001"/>
-    </inertial>
-  </link>
-  <link name="MountToWheel-v1_d">
-    <visual>
-      <origin xyz="0 0 0" rpy="0 0 0"/>
-      <geometry>
-        <mesh filename="package://pfe/meshes/MountToWheel-v1.stl" scale="0.001 0.001 0.001"/>
-      </geometry>
-    </visual>
-    <collision>
-      <origin xyz="0 0 0" rpy="0 0 0"/>
-      <geometry>
-        <mesh filename="package://pfe/meshes/MountToWheel-v1.stl" scale="0.001 0.001 0.001"/>
-      </geometry>
-    </collision>
-    <inertial>
-      <origin xyz="0 0 0" rpy="0 0 0"/>
-      <mass value="0.1"/>
-      <inertia ixx="0.0001" ixy="0" ixz="0" iyy="0.0001" iyz="0" izz="0.0001"/>
-    </inertial>
-  </link>
-  <!-- ===================== WHEEL JOINT LINKS ===================== -->
-  <link name="WheelJoint-v1_a">
-    <visual>
-      <origin xyz="0 0 0" rpy="0 0 0"/>
-      <geometry>
-        <mesh filename="package://pfe/meshes/WheelJoint-v1.stl" scale="0.001 0.001 0.001"/>
-      </geometry>
-    </visual>
-    <collision>
-      <origin xyz="0 0 0" rpy="0 0 0"/>
-      <geometry>
-        <mesh filename="package://pfe/meshes/WheelJoint-v1.stl" scale="0.001 0.001 0.001"/>
-      </geometry>
-    </collision>
-    <inertial>
-      <origin xyz="0 0 0" rpy="0 0 0"/>
-      <mass value="0.05"/>
-      <inertia ixx="0.00005" ixy="0" ixz="0" iyy="0.00005" iyz="0" izz="0.00005"/>
-    </inertial>
-  </link>
-  <link name="WheelJoint-v1_b">
-    <visual>
-      <origin xyz="0 0 0" rpy="0 0 0"/>
-      <geometry>
-        <mesh filename="package://pfe/meshes/WheelJoint-v1.stl" scale="0.001 0.001 0.001"/>
-      </geometry>
-    </visual>
-    <collision>
-      <origin xyz="0 0 0" rpy="0 0 0"/>
-      <geometry>
-        <mesh filename="package://pfe/meshes/WheelJoint-v1.stl" scale="0.001 0.001 0.001"/>
-      </geometry>
-    </collision>
-    <inertial>
-      <origin xyz="0 0 0" rpy="0 0 0"/>
-      <mass value="0.05"/>
-      <inertia ixx="0.00005" ixy="0" ixz="0" iyy="0.00005" iyz="0" izz="0.00005"/>
-    </inertial>
-  </link>
-  <link name="WheelJoint-v1_c">
-    <visual>
-      <origin xyz="0 0 0" rpy="0 0 0"/>
-      <geometry>
-        <mesh filename="package://pfe/meshes/WheelJoint-v1.stl" scale="0.001 0.001 0.001"/>
-      </geometry>
-    </visual>
-    <collision>
-      <origin xyz="0 0 0" rpy="0 0 0"/>
-      <geometry>
-        <mesh filename="package://pfe/meshes/WheelJoint-v1.stl" scale="0.001 0.001 0.001"/>
-      </geometry>
-    </collision>
-    <inertial>
-      <origin xyz="0 0 0" rpy="0 0 0"/>
-      <mass value="0.05"/>
-      <inertia ixx="0.00005" ixy="0" ixz="0" iyy="0.00005" iyz="0" izz="0.00005"/>
-    </inertial>
-  </link>
-  <link name="WheelJoint-v1_d">
-    <visual>
-      <origin xyz="0 0 0" rpy="0 0 0"/>
-      <geometry>
-        <mesh filename="package://pfe/meshes/WheelJoint-v1.stl" scale="0.001 0.001 0.001"/>
-      </geometry>
-    </visual>
-    <collision>
-      <origin xyz="0 0 0" rpy="0 0 0"/>
-      <geometry>
-        <mesh filename="package://pfe/meshes/WheelJoint-v1.stl" scale="0.001 0.001 0.001"/>
-      </geometry>
-    </collision>
-    <inertial>
-      <origin xyz="0 0 0" rpy="0 0 0"/>
-      <mass value="0.05"/>
-      <inertia ixx="0.00005" ixy="0" ixz="0" iyy="0.00005" iyz="0" izz="0.00005"/>
-    </inertial>
-  </link>
-  <!-- ===================== ARDUCAM LINK ===================== -->
+        <mesh filename="package://pfe/meshes/base_link-v3.stl" scale="0.001 0.001 0.001"/>
+      </geometry>
+    </collision>
+  </link>
+  <joint name="base_to_cad" type="fixed">
+    <parent link="base_link"/>
+    <child link="base_cad"/>
+    <origin xyz="0 0 0" rpy="0 0 3.141592653589793"/>
+  </joint>
+  <!-- ===================== WHEELS (MECANUM) ===================== -->
+  <!-- Mapping from your Fusion positions with Fusion axes:
+       front = more negative x  (since +x is backwards)
+       right = more positive y  (since +y is right)
+  -->
+  <link name="front_left_wheel_link">
+    <visual>
+      <geometry>
+        <mesh filename="package://pfe/meshes/wheel_link-v1.stl" scale="0.001 0.001 0.001"/>
+      </geometry>
+    </visual>
+    <collision>
+      <geometry>
+        <mesh filename="package://pfe/meshes/wheel_link-v1.stl" scale="0.001 0.001 0.001"/>
+      </geometry>
+    </collision>
+    <inertial>
+      <origin xyz="2.9766545619658303e-05 4.304267826675812e-06 0.004179545797070823" rpy="0 0 0"/>
+      <mass value="0.3360663312138791"/>
+      <inertia ixx="9.012634603781933e-05" iyy="9.001291913218745e-05" izz="0.00013234115795366513"
+               ixy="1.8834943431300655e-09" iyz="1.41718145309222e-08" ixz="1.2750272517306205e-07"/>
+    </inertial>
+  </link>
+  <link name="rear_left_wheel_link">
+    <visual>
+      <geometry>
+        <mesh filename="package://pfe/meshes/wheel_link-v1.stl" scale="0.001 0.001 0.001"/>
+      </geometry>
+    </visual>
+    <collision>
+      <geometry>
+        <mesh filename="package://pfe/meshes/wheel_link-v1.stl" scale="0.001 0.001 0.001"/>
+      </geometry>
+    </collision>
+    <inertial>
+      <origin xyz="2.9770008680891636e-05 4.304267826675812e-06 0.004179545797070076" rpy="0 0 0"/>
+      <mass value="0.3360663312138791"/>
+      <inertia ixx="9.012634603780545e-05" iyy="9.001291913220827e-05" izz="0.00013234115795369462"
+               ixy="1.8834943587429966e-09" iyz="1.4171814541469944e-08" ixz="1.275027251867153e-07"/>
+    </inertial>
+  </link>
+  <link name="rear_right_wheel_link">
+    <visual>
+      <geometry>
+        <mesh filename="package://pfe/meshes/wheel_link-v1.stl" scale="0.001 0.001 0.001"/>
+      </geometry>
+    </visual>
+    <collision>
+      <geometry>
+        <mesh filename="package://pfe/meshes/wheel_link-v1.stl" scale="0.001 0.001 0.001"/>
+      </geometry>
+    </collision>
+    <inertial>
+      <origin xyz="-2.9768983099991432e-05 -4.304267826960029e-06 0.004179546726436565" rpy="0 0 0"/>
+      <mass value="0.3360663312138791"/>
+      <inertia ixx="9.012634603783667e-05" iyy="9.001291913223602e-05" izz="0.00013234115795369636"
+               ixy="1.883494383896067e-09" iyz="-1.4171814507720273e-08" ixz="-1.2750272519496293e-07"/>
+    </inertial>
+  </link>
+  <link name="front_right_wheel_link">
+    <visual>
+      <geometry>
+        <mesh filename="package://pfe/meshes/wheel_link-v1.stl" scale="0.001 0.001 0.001"/>
+      </geometry>
+    </visual>
+    <collision>
+      <geometry>
+        <mesh filename="package://pfe/meshes/wheel_link-v1.stl" scale="0.001 0.001 0.001"/>
+      </geometry>
+    </collision>
+    <inertial>
+      <origin xyz="-2.9772331126451947e-05 -4.304267826960029e-06 0.0041795467264360096" rpy="0 0 0"/>
+      <mass value="0.3360663312138791"/>
+      <inertia ixx="9.012634603783667e-05" iyy="9.001291913222215e-05" izz="0.00013234115795368248"
+               ixy="1.883494403845387e-09" iyz="-1.4171814508153954e-08" ixz="-1.2750272519626397e-07"/>
+    </inertial>
+  </link>
+  <!-- Wheel joints: parent under base_cad so Fusion transforms remain valid -->
+  <joint name="front_left_wheel_joint" type="continuous">
+    <parent link="base_cad"/>
+    <child link="front_left_wheel_link"/>
+    <origin xyz="-0.2329295352862411 -0.01429999799095302 -0.15665336918407297"
+            rpy="1.5707963267948957 -1.5265566588595922e-16 7.21644966006352e-16"/>
+    <axis xyz="0 0 1"/>
+  </joint>
+  <joint name="rear_left_wheel_joint" type="continuous">
+    <parent link="base_cad"/>
+    <child link="rear_left_wheel_link"/>
+    <origin xyz="-0.10492999528624117 -0.01429999799095293 -0.1566533691840729"
+            rpy="1.5707963267948957 -1.5265566588595922e-16 7.21644966006352e-16"/>
+    <axis xyz="0 0 1"/>
+  </joint>
+  <joint name="rear_right_wheel_joint" type="continuous">
+    <parent link="base_cad"/>
+    <child link="rear_right_wheel_link"/>
+    <origin xyz="-0.10490178528624114 0.23430000200904744 -0.15665336918407313"
+            rpy="-1.5707963267948941 -1.5265566588595922e-16 7.21644966006352e-16"/>
+    <axis xyz="0 0 1"/>
+  </joint>
+  <joint name="front_right_wheel_joint" type="continuous">
+    <parent link="base_cad"/>
+    <child link="front_right_wheel_link"/>
+    <origin xyz="-0.23290132528624108 0.23430000200904733 -0.15665336918407316"
+            rpy="-1.5707963267948974 -1.5265566588595922e-16 7.21644966006352e-16"/>
+    <axis xyz="0 0 1"/>
+  </joint>
+  <!-- ===================== ARM ===================== -->
+  <link name="arm_link">
+    <inertial>
+      <origin xyz="-2.2902735970831146e-07 0.0017334076218106455 0.0365000048213585" rpy="0 0 0"/>
+      <mass value="0.5338474560099968"/>
+      <inertia ixx="0.00022030891025364568" iyy="0.0011328418152016656" izz="0.0009599083468218444"
+               ixy="9.724324401272355e-10" iyz="-5.204170427930421e-18" ixz="-5.898059818321144e-17"/>
+    </inertial>
+    <visual>
+      <origin xyz="9.349037100037094e-10 0.004999995232077037 0.03650000482135752"
+              rpy="1.5707963267948963 1.5707963267948957 0"/>
+      <geometry>
+        <mesh filename="package://pfe/meshes/arm_link-v1.stl" scale="0.001 0.001 0.001"/>
+      </geometry>
+    </visual>
+    <collision>
+      <origin xyz="9.349037100037094e-10 0.004999995232077037 0.03650000482135752"
+              rpy="1.5707963267948963 1.5707963267948957 0"/>
+      <geometry>
+        <mesh filename="package://pfe/meshes/arm_link-v1.stl" scale="0.001 0.001 0.001"/>
+      </geometry>
+    </collision>
+  </link>
+  <joint name="arm_joint" type="continuous">
+    <parent link="base_cad"/>
+    <child link="arm_link"/>
+    <origin xyz="-0.3689156752862411 0.07293206200904699 -0.14265636918407304"
+            rpy="-1.5707963267948974 -1.5265566588595922e-16 7.21644966006352e-16"/>
+    <axis xyz="0 0 1"/>
+  </joint>
+  <!-- ===================== FLIPPER ===================== -->
+  <link name="flipper_link">
+    <inertial>
+      <origin xyz="2.6474475234294913e-09 4.767925592119582e-09 -0.07580524145430977" rpy="0 0 0"/>
+      <mass value="0.4797185340176825"/>
+      <inertia ixx="0.0011969873864993257" iyy="0.0009456324882451857" izz="0.0002533232197152197"
+               ixy="-1.3010426069826053e-18" iyz="1.734723475976807e-18" ixz="1.7802599672211983e-16"/>
+    </inertial>
+    <visual>
+      <origin xyz="0.00861550378970137 0.01247089554740951 -0.07550000482135592"
+              rpy="-1.5707963267948968 -1.5707963267947291 0"/>
+      <geometry>
+        <mesh filename="package://pfe/meshes/flipper_link-v1.stl" scale="0.001 0.001 0.001"/>
+      </geometry>
+    </visual>
+    <collision>
+      <origin xyz="0.00861550378970137 0.01247089554740951 -0.07550000482135592"
+              rpy="-1.5707963267948968 -1.5707963267947291 0"/>
+      <geometry>
+        <mesh filename="package://pfe/meshes/flipper_link-v1.stl" scale="0.001 0.001 0.001"/>
+      </geometry>
+    </collision>
+  </link>
+  <joint name="flipper_joint" type="continuous">
+    <parent link="base_cad"/>
+    <child link="flipper_link"/>
+    <origin xyz="-0.0164154352862412 0.03393206200904719 -0.13965336918407295"
+            rpy="1.5707963267948957 -1.5265566588595922e-16 7.21644966006352e-16"/>
+    <axis xyz="0 0 1"/>
+  </joint>
+  <!-- ===================== CAMERA ===================== -->
   <link name="arducam_link">
-    <visual>
-      <origin xyz="0 0 0" rpy="0 0 0"/>
-      <geometry>
-        <mesh filename="package://pfe/meshes/arducam_link-v1.stl" scale="0.001 0.001 0.001"/>
-      </geometry>
-    </visual>
-    <collision>
-      <origin xyz="0 0 0" rpy="0 0 0"/>
-      <geometry>
-        <mesh filename="package://pfe/meshes/arducam_link-v1.stl" scale="0.001 0.001 0.001"/>
-      </geometry>
-    </collision>
-    <inertial>
-      <origin xyz="0 0 0" rpy="0 0 0"/>
-      <mass value="0.1"/>
-      <inertia ixx="0.0001" ixy="0" ixz="0" iyy="0.0001" iyz="0" izz="0.0001"/>
-    </inertial>
-  </link>
-  <!-- ===================== JOINTS ===================== -->
-  <!-- Base to MountToWheel -->
-  <joint name="base_to_MountToWheel_a" type="fixed">
-    <parent link="base_link"/>
-    <child link="MountToWheel-v1_a"/>
-    <origin xyz="0.163 0.215 0.005" rpy="3.1416 0 3.1416"/>
-  </joint>
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