Commit message: Added suction cups to URDF

File: ws/src/pfe/description/my_robot.urdf.xacro (robot description, xacro)
@@ -11,5 +11,4 @@
   </joint>
   <!-- ===================== CAD WRAPPER (Fusion frame) ===================== -->
-  <!-- Fusion: +x backward, +y right  => rotate CAD frame by pi about Z to match ROS -->
   <link name="base_cad">
     <inertial>
@@ -32,114 +31,9 @@
     </collision>
   </link>
+  <!-- Fusion: +x backward, +y right -->
   <joint name="base_to_cad" type="fixed">
     <parent link="base_link"/>
     <child link="base_cad"/>
     <origin xyz="0 0 0" rpy="0 0 3.141592653589793"/>
-  </joint>
-  <!-- ===================== WHEELS (MECANUM) ===================== -->
-  <!-- Mapping from your Fusion positions with Fusion axes:
-       front = more negative x  (since +x is backwards)
-       right = more positive y  (since +y is right)
-  -->
-  <link name="front_left_wheel_link">
-    <visual>
-      <geometry>
-        <mesh filename="package://pfe/meshes/wheel_link-v1.stl" scale="0.001 0.001 0.001"/>
-      </geometry>
-    </visual>
-    <collision>
-      <geometry>
-        <mesh filename="package://pfe/meshes/wheel_link-v1.stl" scale="0.001 0.001 0.001"/>
-      </geometry>
-    </collision>
-    <inertial>
-      <origin xyz="2.9766545619658303e-05 4.304267826675812e-06 0.004179545797070823" rpy="0 0 0"/>
-      <mass value="0.3360663312138791"/>
-      <inertia ixx="9.012634603781933e-05" iyy="9.001291913218745e-05" izz="0.00013234115795366513"
-               ixy="1.8834943431300655e-09" iyz="1.41718145309222e-08" ixz="1.2750272517306205e-07"/>
-    </inertial>
-  </link>
-  <link name="rear_left_wheel_link">
-    <visual>
-      <geometry>
-        <mesh filename="package://pfe/meshes/wheel_link-v1.stl" scale="0.001 0.001 0.001"/>
-      </geometry>
-    </visual>
-    <collision>
-      <geometry>
-        <mesh filename="package://pfe/meshes/wheel_link-v1.stl" scale="0.001 0.001 0.001"/>
-      </geometry>
-    </collision>
-    <inertial>
-      <origin xyz="2.9770008680891636e-05 4.304267826675812e-06 0.004179545797070076" rpy="0 0 0"/>
-      <mass value="0.3360663312138791"/>
-      <inertia ixx="9.012634603780545e-05" iyy="9.001291913220827e-05" izz="0.00013234115795369462"
-               ixy="1.8834943587429966e-09" iyz="1.4171814541469944e-08" ixz="1.275027251867153e-07"/>
-    </inertial>
-  </link>
-  <link name="rear_right_wheel_link">
-    <visual>
-      <geometry>
-        <mesh filename="package://pfe/meshes/wheel_link-v1.stl" scale="0.001 0.001 0.001"/>
-      </geometry>
-    </visual>
-    <collision>
-      <geometry>
-        <mesh filename="package://pfe/meshes/wheel_link-v1.stl" scale="0.001 0.001 0.001"/>
-      </geometry>
-    </collision>
-    <inertial>
-      <origin xyz="-2.9768983099991432e-05 -4.304267826960029e-06 0.004179546726436565" rpy="0 0 0"/>
-      <mass value="0.3360663312138791"/>
-      <inertia ixx="9.012634603783667e-05" iyy="9.001291913223602e-05" izz="0.00013234115795369636"
-               ixy="1.883494383896067e-09" iyz="-1.4171814507720273e-08" ixz="-1.2750272519496293e-07"/>
-    </inertial>
-  </link>
-  <link name="front_right_wheel_link">
-    <visual>
-      <geometry>
-        <mesh filename="package://pfe/meshes/wheel_link-v1.stl" scale="0.001 0.001 0.001"/>
-      </geometry>
-    </visual>
-    <collision>
-      <geometry>
-        <mesh filename="package://pfe/meshes/wheel_link-v1.stl" scale="0.001 0.001 0.001"/>
-      </geometry>
-    </collision>
-    <inertial>
-      <origin xyz="-2.9772331126451947e-05 -4.304267826960029e-06 0.0041795467264360096" rpy="0 0 0"/>
-      <mass value="0.3360663312138791"/>
-      <inertia ixx="9.012634603783667e-05" iyy="9.001291913222215e-05" izz="0.00013234115795368248"
-               ixy="1.883494403845387e-09" iyz="-1.4171814508153954e-08" ixz="-1.2750272519626397e-07"/>
-    </inertial>
-  </link>
-  <!-- Wheel joints: parent under base_cad so Fusion transforms remain valid -->
-  <joint name="front_left_wheel_joint" type="continuous">
-    <parent link="base_cad"/>
-    <child link="front_left_wheel_link"/>
-    <origin xyz="-0.2329295352862411 -0.01429999799095302 -0.15665336918407297"
-            rpy="1.5707963267948957 -1.5265566588595922e-16 7.21644966006352e-16"/>
-    <axis xyz="0 0 1"/>
-  </joint>
-  <joint name="rear_left_wheel_joint" type="continuous">
-    <parent link="base_cad"/>
-    <child link="rear_left_wheel_link"/>
-    <origin xyz="-0.10492999528624117 -0.01429999799095293 -0.1566533691840729"
-            rpy="1.5707963267948957 -1.5265566588595922e-16 7.21644966006352e-16"/>
-    <axis xyz="0 0 1"/>
-  </joint>
-  <joint name="rear_right_wheel_joint" type="continuous">
-    <parent link="base_cad"/>
-    <child link="rear_right_wheel_link"/>
-    <origin xyz="-0.10490178528624114 0.23430000200904744 -0.15665336918407313"
-            rpy="-1.5707963267948941 -1.5265566588595922e-16 7.21644966006352e-16"/>
-    <axis xyz="0 0 1"/>
-  </joint>
-  <joint name="front_right_wheel_joint" type="continuous">
-    <parent link="base_cad"/>
-    <child link="front_right_wheel_link"/>
-    <origin xyz="-0.23290132528624108 0.23430000200904733 -0.15665336918407316"
-            rpy="-1.5707963267948974 -1.5265566588595922e-16 7.21644966006352e-16"/>
-    <axis xyz="0 0 1"/>
   </joint>
   <!-- ===================== ARM ===================== -->
@@ -203,12 +97,51 @@
     <axis xyz="0 0 1"/>
   </joint>
+  <!-- ===================== MECANUM WHEELS ===================== -->
+  <link name="front_left_wheel_link">
+    <visual><geometry><mesh filename="package://pfe/meshes/wheel_link-v1.stl" scale="0.001 0.001 0.001"/></geometry></visual>
+    <collision><geometry><mesh filename="package://pfe/meshes/wheel_link-v1.stl" scale="0.001 0.001 0.001"/></geometry></collision>
+  </link>
+  <link name="rear_left_wheel_link">
+    <visual><geometry><mesh filename="package://pfe/meshes/wheel_link-v1.stl" scale="0.001 0.001 0.001"/></geometry></visual>
+    <collision><geometry><mesh filename="package://pfe/meshes/wheel_link-v1.stl" scale="0.001 0.001 0.001"/></geometry></collision>
+  </link>
+  <link name="rear_right_wheel_link">
+    <visual><geometry><mesh filename="package://pfe/meshes/wheel_link-v1.stl" scale="0.001 0.001 0.001"/></geometry></visual>
+    <collision><geometry><mesh filename="package://pfe/meshes/wheel_link-v1.stl" scale="0.001 0.001 0.001"/></geometry></collision>
+  </link>
+  <link name="front_right_wheel_link">
+    <visual><geometry><mesh filename="package://pfe/meshes/wheel_link-v1.stl" scale="0.001 0.001 0.001"/></geometry></visual>
+    <collision><geometry><mesh filename="package://pfe/meshes/wheel_link-v1.stl" scale="0.001 0.001 0.001"/></geometry></collision>
+  </link>
+  <joint name="front_left_wheel_joint" type="continuous">
+    <parent link="base_cad"/>
+    <child link="front_left_wheel_link"/>
+    <origin xyz="-0.2329295352862411 -0.01429999799095302 -0.15665336918407297"
+            rpy="1.5707963267948957 -1.5265566588595922e-16 7.21644966006352e-16"/>
+    <axis xyz="0 0 1"/>
+  </joint>
+  <joint name="rear_left_wheel_joint" type="continuous">
+    <parent link="base_cad"/>
+    <child link="rear_left_wheel_link"/>
+    <origin xyz="-0.10492999528624117 -0.01429999799095293 -0.1566533691840729"
+            rpy="1.5707963267948957 -1.5265566588595922e-16 7.21644966006352e-16"/>
+    <axis xyz="0 0 1"/>
+  </joint>
+  <joint name="rear_right_wheel_joint" type="continuous">
+    <parent link="base_cad"/>
+    <child link="rear_right_wheel_link"/>
+    <origin xyz="-0.10490178528624114 0.23430000200904744 -0.15665336918407313"
+            rpy="-1.5707963267948941 -1.5265566588595922e-16 7.21644966006352e-16"/>
+    <axis xyz="0 0 1"/>
+  </joint>
+  <joint name="front_right_wheel_joint" type="continuous">
+    <parent link="base_cad"/>
+    <child link="front_right_wheel_link"/>
+    <origin xyz="-0.23290132528624108 0.23430000200904733 -0.15665336918407316"
+            rpy="-1.5707963267948974 -1.5265566588595922e-16 7.21644966006352e-16"/>
+    <axis xyz="0 0 1"/>
+  </joint>
   <!-- ===================== CAMERA ===================== -->
   <link name="arducam_link">
-    <inertial>
-      <origin xyz="0.00013322309970456914 -0.000950447708985589 0.00043137326239044426" rpy="0 0 0"/>
-      <mass value="0.0010174438167060709"/>
-      <inertia ixx="4.5307132551573865e-08" iyy="3.509024203284948e-08" izz="7.596114417939664e-08"
-               ixy="1.0347644394365709e-09" iyz="2.2640703271659043e-09" ixz="-1.316658641836537e-10"/>
-    </inertial>
     <visual>
       <origin xyz="1.7220046188981542e-09 4.813011891258156e-09 -0.0017500015693401494"
@@ -232,3 +165,42 @@
             rpy="-3.141592653589791 -1.178097245096172 -3.141592653589791"/>
   </joint>
+  <!-- ===================== SUCTION CUPS ===================== -->
+  <!-- arm_link IS the intake bar -->
+  <link name="cup_0">
+    <visual><geometry><mesh filename="package://pfe/meshes/suctioncup_link-v1.stl" scale="0.001 0.001 0.001"/></geometry></visual>
+    <collision><geometry><mesh filename="package://pfe/meshes/suctioncup_link-v1.stl" scale="0.001 0.001 0.001"/></geometry></collision>
+  </link>
+  <link name="cup_1">
+    <visual><geometry><mesh filename="package://pfe/meshes/suctioncup_link-v1.stl" scale="0.001 0.001 0.001"/></geometry></visual>
+    <collision><geometry><mesh filename="package://pfe/meshes/suctioncup_link-v1.stl" scale="0.001 0.001 0.001"/></geometry></collision>
+  </link>
+  <link name="cup_2">
+    <visual><geometry><mesh filename="package://pfe/meshes/suctioncup_link-v1.stl" scale="0.001 0.001 0.001"/></geometry></visual>
+    <collision><geometry><mesh filename="package://pfe/meshes/suctioncup_link-v1.stl" scale="0.001 0.001 0.001"/></geometry></collision>
+  </link>
+  <link name="cup_3">
+    <visual><geometry><mesh filename="package://pfe/meshes/suctioncup_link-v1.stl" scale="0.001 0.001 0.001"/></geometry></visual>
+    <collision><geometry><mesh filename="package://pfe/meshes/suctioncup_link-v1.stl" scale="0.001 0.001 0.001"/></geometry></collision>
+  </link>
+  <!-- Keep your exact fixed transforms -->
+  <joint name="arm_to_cup_0" type="fixed">
+    <parent link="arm_link"/>
+    <child link="cup_0"/>
+    <origin xyz="0.075 0.0105 0.0365" rpy="1.5707963267948966 0 0"/>
+  </joint>
+  <joint name="arm_to_cup_1" type="fixed">
+    <parent link="arm_link"/>
+    <child link="cup_1"/>
+    <origin xyz="0.025 0.0100 0.0365" rpy="-1.5707963267948966 0 0"/>
+  </joint>
+  <joint name="arm_to_cup_2" type="fixed">
+    <parent link="arm_link"/>
+    <child link="cup_2"/>
+    <origin xyz="-0.025 0.0105 0.0365" rpy="1.5707963267948966 0 0"/>
+  </joint>
+  <joint name="arm_to_cup_3" type="fixed">
+    <parent link="arm_link"/>
+    <child link="cup_3"/>
+    <origin xyz="-0.075 0.0105 0.0365" rpy="1.5707963267948966 0 0"/>
+  </joint>
 </robot>

Commit message: URDF change for new camera position

File: ws/src/pfe/description/my_robot.urdf.xacro (robot description, xacro)
@@ -10,16 +10,16 @@
     <origin xyz="0 0 0" rpy="0 0 0"/>
   </joint>
-  <!-- ===================== CAD WRAPPER (Fusion frame) ===================== -->
+  <!-- ===================== CAD WRAPPER ===================== -->
   <link name="base_cad">
     <inertial>
-      <origin xyz="-0.181130474842482 0.10958995900517023 -0.10051074270429218" rpy="0 0 0"/>
-      <mass value="10.802255131301344"/>
-      <inertia ixx="0.11142549471720897" iyy="0.15234586542751433" izz="0.15214678916514196"
-               ixy="0.0002653832816470656" iyz="0.00027410838368888666" ixz="0.009773387741291757"/>
+      <origin xyz="-0.1806532478764334 0.10959136535685834 -0.09958100133613353" rpy="0 0 0"/>
+      <mass value="10.846844826170994"/>
+      <inertia ixx="0.1137300898429841" iyy="0.15506270343665957" izz="0.1525596007466387"
+               ixy="0.0002636196730894534" iyz="0.0002706724915273537" ixz="0.008689234245133912"/>
     </inertial>
     <visual>
       <origin xyz="0 0 0" rpy="0 0 0"/>
       <geometry>
-        <mesh filename="package://pfe/meshes/base_link-v3.stl" scale="0.001 0.001 0.001"/>
+        <mesh filename="package://pfe/meshes/base_link-v5.stl" scale="0.001 0.001 0.001"/>
       </geometry>
     </visual>
@@ -27,5 +27,5 @@
       <origin xyz="0 0 0" rpy="0 0 0"/>
       <geometry>
-        <mesh filename="package://pfe/meshes/base_link-v3.stl" scale="0.001 0.001 0.001"/>
+        <mesh filename="package://pfe/meshes/base_link-v5.stl" scale="0.001 0.001 0.001"/>
       </geometry>
     </collision>
@@ -99,18 +99,50 @@
   <!-- ===================== MECANUM WHEELS ===================== -->
   <link name="front_left_wheel_link">
-    <visual><geometry><mesh filename="package://pfe/meshes/wheel_link-v1.stl" scale="0.001 0.001 0.001"/></geometry></visual>
-    <collision><geometry><mesh filename="package://pfe/meshes/wheel_link-v1.stl" scale="0.001 0.001 0.001"/></geometry></collision>
+    <visual>
+      <geometry>
+        <mesh filename="package://pfe/meshes/wheel_link-v1.stl" scale="0.001 0.001 0.001"/>
+      </geometry>
+    </visual>
+    <collision>
+      <geometry>
+        <mesh filename="package://pfe/meshes/wheel_link-v1.stl" scale="0.001 0.001 0.001"/>
+      </geometry>
+    </collision>
   </link>
   <link name="rear_left_wheel_link">
-    <visual><geometry><mesh filename="package://pfe/meshes/wheel_link-v1.stl" scale="0.001 0.001 0.001"/></geometry></visual>
-    <collision><geometry><mesh filename="package://pfe/meshes/wheel_link-v1.stl" scale="0.001 0.001 0.001"/></geometry></collision>
+    <visual>
+      <geometry>
+        <mesh filename="package://pfe/meshes/wheel_link-v1.stl" scale="0.001 0.001 0.001"/>
+      </geometry>
+    </visual>
+    <collision>
+      <geometry>
+        <mesh filename="package://pfe/meshes/wheel_link-v1.stl" scale="0.001 0.001 0.001"/>
+      </geometry>
+    </collision>
   </link>
   <link name="rear_right_wheel_link">
-    <visual><geometry><mesh filename="package://pfe/meshes/wheel_link-v1.stl" scale="0.001 0.001 0.001"/></geometry></visual>
-    <collision><geometry><mesh filename="package://pfe/meshes/wheel_link-v1.stl" scale="0.001 0.001 0.001"/></geometry></collision>
+    <visual>
+      <geometry>
+        <mesh filename="package://pfe/meshes/wheel_link-v1.stl" scale="0.001 0.001 0.001"/>
+      </geometry>
+    </visual>
+    <collision>
+      <geometry>
+        <mesh filename="package://pfe/meshes/wheel_link-v1.stl" scale="0.001 0.001 0.001"/>
+      </geometry>
+    </collision>
   </link>
   <link name="front_right_wheel_link">
-    <visual><geometry><mesh filename="package://pfe/meshes/wheel_link-v1.stl" scale="0.001 0.001 0.001"/></geometry></visual>
-    <collision><geometry><mesh filename="package://pfe/meshes/wheel_link-v1.stl" scale="0.001 0.001 0.001"/></geometry></collision>
+    <visual>
+      <geometry>
+        <mesh filename="package://pfe/meshes/wheel_link-v1.stl" scale="0.001 0.001 0.001"/>
+      </geometry>
+    </visual>
+    <collision>
+      <geometry>
+        <mesh filename="package://pfe/meshes/wheel_link-v1.stl" scale="0.001 0.001 0.001"/>
+      </geometry>
+    </collision>
   </link>
   <joint name="front_left_wheel_joint" type="continuous">
@@ -144,7 +176,13 @@
   <!-- ===================== CAMERA ===================== -->
   <link name="arducam_link">
-    <visual>
-      <origin xyz="1.7220046188981542e-09 4.813011891258156e-09 -0.0017500015693401494"
-              rpy="4.31077779183057e-16 1.6653345369377346e-16 -3.1415926535897927"/>
+    <inertial>
+      <origin xyz="-0.00013322161290098224 0.0009504573350092649 0.00043137020324471645" rpy="0 0 0"/>
+      <mass value="0.0010174438167060709"/>
+      <inertia ixx="4.5307132551562007e-08" iyy="3.5090242032863035e-08" izz="7.59611441794051e-08"
+               ixy="1.0347644394329782e-09" iyz="-2.264070327162072e-09" ixz="1.3166586418150303e-10"/>
+    </inertial>
+    <visual>
+      <origin xyz="-2.352010142203653e-10 4.813011784676747e-09 -0.001750004628485895"
+              rpy="8.52607141014584e-18 -5.5511151231257815e-17 9.485990215114392e-16"/>
       <geometry>
         <mesh filename="package://pfe/meshes/arducam_link-v3.stl" scale="0.001 0.001 0.001"/>
@@ -152,6 +190,6 @@
     </visual>
     <collision>
-      <origin xyz="1.7220046188981542e-09 4.813011891258156e-09 -0.0017500015693401494"
-              rpy="4.31077779183057e-16 1.6653345369377346e-16 -3.1415926535897927"/>
+      <origin xyz="-2.352010142203653e-10 4.813011784676747e-09 -0.001750004628485895"
+              rpy="8.52607141014584e-18 -5.5511151231257815e-17 9.485990215114392e-16"/>
       <geometry>
         <mesh filename="package://pfe/meshes/arducam_link-v3.stl" scale="0.001 0.001 0.001"/>
@@ -162,26 +200,56 @@
     <parent link="base_cad"/>
     <child link="arducam_link"/>
-    <origin xyz="-0.21195906528624112 0.10993206200904702 0.0426585308159267"
-            rpy="-3.141592653589791 -1.178097245096172 -3.141592653589791"/>
+    <origin xyz="-0.10964196528624118 0.10993206200904702 0.15264326081592658"
+            rpy="-3.1415926535897922 -0.6973907898697068 -3.141592653589792"/>
   </joint>
   <!-- ===================== SUCTION CUPS ===================== -->
-  <!-- arm_link IS the intake bar -->
   <link name="cup_0">
-    <visual><geometry><mesh filename="package://pfe/meshes/suctioncup_link-v1.stl" scale="0.001 0.001 0.001"/></geometry></visual>
-    <collision><geometry><mesh filename="package://pfe/meshes/suctioncup_link-v1.stl" scale="0.001 0.001 0.001"/></geometry></collision>
+    <visual>
+      <geometry>
+        <mesh filename="package://pfe/meshes/suctioncup_link-v1.stl" scale="0.001 0.001 0.001"/>
+      </geometry>
+    </visual>
+    <collision>
+      <geometry>
+        <mesh filename="package://pfe/meshes/suctioncup_link-v1.stl" scale="0.001 0.001 0.001"/>
+      </geometry>
+    </collision>
   </link>
   <link name="cup_1">
-    <visual><geometry><mesh filename="package://pfe/meshes/suctioncup_link-v1.stl" scale="0.001 0.001 0.001"/></geometry></visual>
-    <collision><geometry><mesh filename="package://pfe/meshes/suctioncup_link-v1.stl" scale="0.001 0.001 0.001"/></geometry></collision>
+    <visual>
+      <geometry>
+        <mesh filename="package://pfe/meshes/suctioncup_link-v1.stl" scale="0.001 0.001 0.001"/>
+      </geometry>
+    </visual>
+    <collision>
+      <geometry>
+        <mesh filename="package://pfe/meshes/suctioncup_link-v1.stl" scale="0.001 0.001 0.001"/>
+      </geometry>
+    </collision>
   </link>
   <link name="cup_2">
-    <visual><geometry><mesh filename="package://pfe/meshes/suctioncup_link-v1.stl" scale="0.001 0.001 0.001"/></geometry></visual>
-    <collision><geometry><mesh filename="package://pfe/meshes/suctioncup_link-v1.stl" scale="0.001 0.001 0.001"/></geometry></collision>
+    <visual>
+      <geometry>
+        <mesh filename="package://pfe/meshes/suctioncup_link-v1.stl" scale="0.001 0.001 0.001"/>
+      </geometry>
+    </visual>
+    <collision>
+      <geometry>
+        <mesh filename="package://pfe/meshes/suctioncup_link-v1.stl" scale="0.001 0.001 0.001"/>
+      </geometry>
+    </collision>
   </link>
   <link name="cup_3">
-    <visual><geometry><mesh filename="package://pfe/meshes/suctioncup_link-v1.stl" scale="0.001 0.001 0.001"/></geometry></visual>
-    <collision><geometry><mesh filename="package://pfe/meshes/suctioncup_link-v1.stl" scale="0.001 0.001 0.001"/></geometry></collision>
-  </link>
-  <!-- Keep your exact fixed transforms -->
+    <visual>
+      <geometry>
+        <mesh filename="package://pfe/meshes/suctioncup_link-v1.stl" scale="0.001 0.001 0.001"/>
+      </geometry>
+    </visual>
+    <collision>
+      <geometry>
+        <mesh filename="package://pfe/meshes/suctioncup_link-v1.stl" scale="0.001 0.001 0.001"/>
+      </geometry>
+    </collision>
+  </link>
   <joint name="arm_to_cup_0" type="fixed">
     <parent link="arm_link"/>

Commit message: urdf fix for camera

File: ws/src/pfe/description/my_robot.urdf.xacro (robot description, xacro)
@@ -203,4 +203,11 @@
             rpy="-3.1415926535897922 -0.6973907898697068 -3.141592653589792"/>
   </joint>
+  <!-- ROS optical frame for camera-based vision -->
+  <link name="arducam_optical_frame"/>
+  <joint name="arducam_to_optical" type="fixed">
+    <parent link="arducam_link"/>
+    <child link="arducam_optical_frame"/>
+    <origin xyz="0 0 0" rpy="-1.57079632679 0 -1.57079632679"/>
+  </joint>
   <!-- ===================== SUCTION CUPS ===================== -->
   <link name="cup_0">
