Commit message: strategy reorganization + attempted fixes

File: server_ws/src/match/description/my_robot.urdf.xacro (robot description, xacro)
@@ -14,5 +14,5 @@
       <origin xyz="0 0 0" rpy="0 0 0"/>
       <geometry>
-        <mesh filename="package://pfe/meshes/base_link-v5.stl" scale="0.001 0.001 0.001"/>
+        <mesh filename="package://match/meshes/base_link-v5.stl" scale="0.001 0.001 0.001"/>
       </geometry>
     </visual>
@@ -20,5 +20,5 @@
       <origin xyz="0 0 0" rpy="0 0 0"/>
       <geometry>
-        <mesh filename="package://pfe/meshes/base_link-v5.stl" scale="0.001 0.001 0.001"/>
+        <mesh filename="package://match/meshes/base_link-v5.stl" scale="0.001 0.001 0.001"/>
       </geometry>
     </collision>
@@ -42,5 +42,5 @@
               rpy="1.5707963267948963 1.5707963267948957 0"/>
       <geometry>
-        <mesh filename="package://pfe/meshes/arm_link-v1.stl" scale="0.001 0.001 0.001"/>
+        <mesh filename="package://match/meshes/arm_link-v1.stl" scale="0.001 0.001 0.001"/>
       </geometry>
     </visual>
@@ -49,5 +49,5 @@
               rpy="1.5707963267948963 1.5707963267948957 0"/>
       <geometry>
-        <mesh filename="package://pfe/meshes/arm_link-v1.stl" scale="0.001 0.001 0.001"/>
+        <mesh filename="package://match/meshes/arm_link-v1.stl" scale="0.001 0.001 0.001"/>
       </geometry>
     </collision>
@@ -72,5 +72,5 @@
               rpy="-1.5707963267948968 -1.5707963267947291 0"/>
       <geometry>
-        <mesh filename="package://pfe/meshes/flipper_link-v1.stl" scale="0.001 0.001 0.001"/>
+        <mesh filename="package://match/meshes/flipper_link-v1.stl" scale="0.001 0.001 0.001"/>
       </geometry>
     </visual>
@@ -79,5 +79,5 @@
               rpy="-1.5707963267948968 -1.5707963267947291 0"/>
       <geometry>
-        <mesh filename="package://pfe/meshes/flipper_link-v1.stl" scale="0.001 0.001 0.001"/>
+        <mesh filename="package://match/meshes/flipper_link-v1.stl" scale="0.001 0.001 0.001"/>
       </geometry>
     </collision>
@@ -94,10 +94,10 @@
     <visual>
       <geometry>
-        <mesh filename="package://pfe/meshes/wheel_link-v1.stl" scale="0.001 0.001 0.001"/>
-      </geometry>
-    </visual>
-    <collision>
-      <geometry>
-        <mesh filename="package://pfe/meshes/wheel_link-v1.stl" scale="0.001 0.001 0.001"/>
+        <mesh filename="package://match/meshes/wheel_link-v1.stl" scale="0.001 0.001 0.001"/>
+      </geometry>
+    </visual>
+    <collision>
+      <geometry>
+        <mesh filename="package://match/meshes/wheel_link-v1.stl" scale="0.001 0.001 0.001"/>
       </geometry>
     </collision>
@@ -106,10 +106,10 @@
     <visual>
       <geometry>
-        <mesh filename="package://pfe/meshes/wheel_link-v1.stl" scale="0.001 0.001 0.001"/>
-      </geometry>
-    </visual>
-    <collision>
-      <geometry>
-        <mesh filename="package://pfe/meshes/wheel_link-v1.stl" scale="0.001 0.001 0.001"/>
+        <mesh filename="package://match/meshes/wheel_link-v1.stl" scale="0.001 0.001 0.001"/>
+      </geometry>
+    </visual>
+    <collision>
+      <geometry>
+        <mesh filename="package://match/meshes/wheel_link-v1.stl" scale="0.001 0.001 0.001"/>
       </geometry>
     </collision>
@@ -118,10 +118,10 @@
     <visual>
       <geometry>
-        <mesh filename="package://pfe/meshes/wheel_link-v1.stl" scale="0.001 0.001 0.001"/>
-      </geometry>
-    </visual>
-    <collision>
-      <geometry>
-        <mesh filename="package://pfe/meshes/wheel_link-v1.stl" scale="0.001 0.001 0.001"/>
+        <mesh filename="package://match/meshes/wheel_link-v1.stl" scale="0.001 0.001 0.001"/>
+      </geometry>
+    </visual>
+    <collision>
+      <geometry>
+        <mesh filename="package://match/meshes/wheel_link-v1.stl" scale="0.001 0.001 0.001"/>
       </geometry>
     </collision>
@@ -130,10 +130,10 @@
     <visual>
       <geometry>
-        <mesh filename="package://pfe/meshes/wheel_link-v1.stl" scale="0.001 0.001 0.001"/>
-      </geometry>
-    </visual>
-    <collision>
-      <geometry>
-        <mesh filename="package://pfe/meshes/wheel_link-v1.stl" scale="0.001 0.001 0.001"/>
+        <mesh filename="package://match/meshes/wheel_link-v1.stl" scale="0.001 0.001 0.001"/>
+      </geometry>
+    </visual>
+    <collision>
+      <geometry>
+        <mesh filename="package://match/meshes/wheel_link-v1.stl" scale="0.001 0.001 0.001"/>
       </geometry>
     </collision>
@@ -179,5 +179,5 @@
               rpy="8.52607141014584e-18 -5.5511151231257815e-17 9.485990215114392e-16"/>
       <geometry>
-        <mesh filename="package://pfe/meshes/arducam_link-v3.stl" scale="0.001 0.001 0.001"/>
+        <mesh filename="package://match/meshes/arducam_link-v3.stl" scale="0.001 0.001 0.001"/>
       </geometry>
     </visual>
@@ -186,5 +186,5 @@
               rpy="8.52607141014584e-18 -5.5511151231257815e-17 9.485990215114392e-16"/>
       <geometry>
-        <mesh filename="package://pfe/meshes/arducam_link-v3.stl" scale="0.001 0.001 0.001"/>
+        <mesh filename="package://match/meshes/arducam_link-v3.stl" scale="0.001 0.001 0.001"/>
       </geometry>
     </collision>
@@ -207,10 +207,10 @@
     <visual>
       <geometry>
-        <mesh filename="package://pfe/meshes/suctioncup_link-v1.stl" scale="0.001 0.001 0.001"/>
-      </geometry>
-    </visual>
-    <collision>
-      <geometry>
-        <mesh filename="package://pfe/meshes/suctioncup_link-v1.stl" scale="0.001 0.001 0.001"/>
+        <mesh filename="package://match/meshes/suctioncup_link-v1.stl" scale="0.001 0.001 0.001"/>
+      </geometry>
+    </visual>
+    <collision>
+      <geometry>
+        <mesh filename="package://match/meshes/suctioncup_link-v1.stl" scale="0.001 0.001 0.001"/>
       </geometry>
     </collision>
@@ -219,10 +219,10 @@
     <visual>
       <geometry>
-        <mesh filename="package://pfe/meshes/suctioncup_link-v1.stl" scale="0.001 0.001 0.001"/>
-      </geometry>
-    </visual>
-    <collision>
-      <geometry>
-        <mesh filename="package://pfe/meshes/suctioncup_link-v1.stl" scale="0.001 0.001 0.001"/>
+        <mesh filename="package://match/meshes/suctioncup_link-v1.stl" scale="0.001 0.001 0.001"/>
+      </geometry>
+    </visual>
+    <collision>
+      <geometry>
+        <mesh filename="package://match/meshes/suctioncup_link-v1.stl" scale="0.001 0.001 0.001"/>
       </geometry>
     </collision>
@@ -231,10 +231,10 @@
     <visual>
       <geometry>
-        <mesh filename="package://pfe/meshes/suctioncup_link-v1.stl" scale="0.001 0.001 0.001"/>
-      </geometry>
-    </visual>
-    <collision>
-      <geometry>
-        <mesh filename="package://pfe/meshes/suctioncup_link-v1.stl" scale="0.001 0.001 0.001"/>
+        <mesh filename="package://match/meshes/suctioncup_link-v1.stl" scale="0.001 0.001 0.001"/>
+      </geometry>
+    </visual>
+    <collision>
+      <geometry>
+        <mesh filename="package://match/meshes/suctioncup_link-v1.stl" scale="0.001 0.001 0.001"/>
       </geometry>
     </collision>
@@ -243,10 +243,10 @@
     <visual>
       <geometry>
-        <mesh filename="package://pfe/meshes/suctioncup_link-v1.stl" scale="0.001 0.001 0.001"/>
-      </geometry>
-    </visual>
-    <collision>
-      <geometry>
-        <mesh filename="package://pfe/meshes/suctioncup_link-v1.stl" scale="0.001 0.001 0.001"/>
+        <mesh filename="package://match/meshes/suctioncup_link-v1.stl" scale="0.001 0.001 0.001"/>
+      </geometry>
+    </visual>
+    <collision>
+      <geometry>
+        <mesh filename="package://match/meshes/suctioncup_link-v1.stl" scale="0.001 0.001 0.001"/>
       </geometry>
     </collision>
@@ -272,64 +272,3 @@
     <origin xyz="-0.075 0.0105 0.0365" rpy="1.5707963267948966 0 0"/>
   </joint>
-  <!-- ===================== DEADWHEEL ODOMETRY ===================== -->
-  <link name="deadwheel_right">
-    <visual>
-      <origin xyz="-0.01366075454561134 0 0" rpy="3.1415926535897927 -1.5707963267948957 0"/>
-      <geometry>
-        <mesh filename="package://pfe/meshes/deadwheel_link-v1.stl" scale="0.001 0.001 0.001"/>
-      </geometry>
-    </visual>
-    <collision>
-      <origin xyz="-0.01366075454561134 0 0" rpy="3.1415926535897927 -1.5707963267948957 0"/>
-      <geometry>
-        <mesh filename="package://pfe/meshes/deadwheel_link-v1.stl" scale="0.001 0.001 0.001"/>
-      </geometry>
-    </collision>
-  </link>
-  <link name="deadwheel_left">
-    <visual>
-      <origin xyz="0 0 0.01741075143684732" rpy="0 0 0"/>
-      <geometry>
-        <mesh filename="package://pfe/meshes/deadwheel_link-v1.stl" scale="0.001 0.001 0.001"/>
-      </geometry>
-    </visual>
-    <collision>
-      <origin xyz="0 0 0.01741075143684732" rpy="0 0 0"/>
-      <geometry>
-        <mesh filename="package://pfe/meshes/deadwheel_link-v1.stl" scale="0.001 0.001 0.001"/>
-      </geometry>
-    </collision>
-  </link>
-  <link name="deadwheel_side">
-    <visual>
-      <origin xyz="0 0 -0.018660747990952988" rpy="0 0 0"/>
-      <geometry>
-        <mesh filename="package://pfe/meshes/deadwheel_link-v1.stl" scale="0.001 0.001 0.001"/>
-      </geometry>
-    </visual>
-    <collision>
-      <origin xyz="0 0 -0.018660747990952988" rpy="0 0 0"/>
-      <geometry>
-        <mesh filename="package://pfe/meshes/deadwheel_link-v1.stl" scale="0.001 0.001 0.001"/>
-      </geometry>
-    </collision>
-  </link>
-  <joint name="base_to_deadwheel_right" type="continuous">
-    <parent link="base_cad"/>
-    <child link="deadwheel_right"/>
-    <origin xyz="-0.1689 0.1848 0.0072" rpy="1.57079632679 0 3.14159265359"/>
-    <axis xyz="0 0 -1"/>
-  </joint>
-  <joint name="base_to_deadwheel_left" type="continuous">
-    <parent link="base_cad"/>
-    <child link="deadwheel_left"/>
-    <origin xyz="-0.1689 0.0352 0.0072" rpy="1.57079632679 0 3.14159265359"/>
-    <axis xyz="0 0 -1"/>
-  </joint>
-  <joint name="base_to_deadwheel_side" type="continuous">
-    <parent link="base_cad"/>
-    <child link="deadwheel_side"/>
-    <origin xyz="-0.1059 0.1100 0.0072" rpy="1.57079632679 0 -1.57079632679"/>
-    <axis xyz="-1 0 0"/>
-  </joint>
 </robot>

Commit message: New RUFD!!!

File: server_ws/src/match/description/my_robot.urdf.xacro (robot description, xacro)
@@ -193,5 +193,5 @@
     <parent link="base_cad"/>
     <child link="arducam_link"/>
-    <origin xyz="-0.10964196528624118 0.10993206200904702 0.15264326081592658"
+    <origin xyz="-0.2678761652862411 0.16593206200904703 0.06147094081592663"
             rpy="-3.1415926535897922 -0.6973907898697068 -3.141592653589792"/>
   </joint>

Commit message: urdf

File: server_ws/src/match/description/my_robot.urdf.xacro (robot description, xacro)
@@ -56,5 +56,5 @@
     <parent link="base_cad"/>
     <child link="arm_link"/>
-    <origin xyz="-0.3689156752862411 0.07293206200904699 -0.14265636918407304"
+    <origin xyz="-0.3919156752862411 0.08793206200904699 -0.14265636918407304"
             rpy="-1.5707963267948974 -1.5265566588595922e-16 7.21644966006352e-16"/>
     <axis xyz="0 0 1"/>
@@ -255,20 +255,20 @@
     <parent link="arm_link"/>
     <child link="cup_0"/>
-    <origin xyz="0.075 0.0105 0.0365" rpy="1.5707963267948966 0 0"/>
+    <origin xyz="0.125 0.0105 0.0365" rpy="1.5707963267948966 0 0"/>
   </joint>
   <joint name="arm_to_cup_1" type="fixed">
     <parent link="arm_link"/>
     <child link="cup_1"/>
-    <origin xyz="0.025 0.0100 0.0365" rpy="-1.5707963267948966 0 0"/>
+    <origin xyz="0.075 0.0100 0.0365" rpy="-1.5707963267948966 0 0"/>
   </joint>
   <joint name="arm_to_cup_2" type="fixed">
     <parent link="arm_link"/>
     <child link="cup_2"/>
+    <origin xyz="0.025 0.0105 0.0365" rpy="1.5707963267948966 0 0"/>
+  </joint>
+  <joint name="arm_to_cup_3" type="fixed">
+    <parent link="arm_link"/>
+    <child link="cup_3"/>
     <origin xyz="-0.025 0.0105 0.0365" rpy="1.5707963267948966 0 0"/>
   </joint>
-  <joint name="arm_to_cup_3" type="fixed">
-    <parent link="arm_link"/>
-    <child link="cup_3"/>
-    <origin xyz="-0.075 0.0105 0.0365" rpy="1.5707963267948966 0 0"/>
-  </joint>
 </robot>

Commit message: awd

File: server_ws/src/match/description/my_robot.urdf.xacro (robot description, xacro)
@@ -54,5 +54,5 @@
   </link>
   <joint name="arm_joint" type="continuous">
-    <parent link="base_cad"/>
+    <parent link="base_link"/>
     <child link="arm_link"/>
     <origin xyz="-0.3919156752862411 0.08793206200904699 -0.14265636918407304"

Commit message: wad

File: server_ws/src/match/description/my_robot.urdf.xacro (robot description, xacro)
@@ -6,8 +6,12 @@
   <link name="base_cad">
     <inertial>
-      <origin xyz="-0.1806532478764334 0.10959136535685834 -0.09958100133613353" rpy="0 0 0"/>
-      <mass value="10.846844826170994"/>
-      <inertia ixx="0.1137300898429841" iyy="0.15506270343665957" izz="0.1525596007466387"
-               ixy="0.0002636196730894534" iyz="0.0002706724915273537" ixz="0.008689234245133912"/>
+      <origin xyz="-0.18129580587395977 0.11002670866229906 -0.09830960898232394" rpy="0 0 0"/>
+      <mass value="10.931310813599758"/>
+      <inertia ixx="0.1162758217320149"
+               iyy="0.15792001930992816"
+               izz="0.15341594762610528"
+               ixy="0.0006562989752065123"
+               iyz="-0.0005062993369034275"
+               ixz="0.009839529045043937"/>
     </inertial>
     <visual>
@@ -24,5 +28,5 @@
     </collision>
   </link>
-  <!-- Fusion: +x backward, +y right. Origin offset centers base_link on the robot's wheel centre. -->
+  <!-- Fusion: +x backward, +y right -->
   <joint name="base_to_cad" type="fixed">
     <parent link="base_link"/>
@@ -33,9 +37,14 @@
   <link name="arm_link">
     <inertial>
-      <origin xyz="-2.2902735970831146e-07 0.0017334076218106455 0.0365000048213585" rpy="0 0 0"/>
+      <origin xyz="-9.798976132702034e-16 -2.2996226341901397e-07 0.003266587610266396" rpy="0 0 0"/>
       <mass value="0.5338474560099968"/>
-      <inertia ixx="0.00022030891025364568" iyy="0.0011328418152016656" izz="0.0009599083468218444"
-               ixy="9.724324401272355e-10" iyz="-5.204170427930421e-18" ixz="-5.898059818321144e-17"/>
-    </inertial>
+      <inertia ixx="0.0009599083468218418"
+               iyy="0.0002203089102536459"
+               izz="0.0011328418152016686"
+               ixy="5.970780693414603e-17"
+               iyz="-9.724324403256641e-10"
+               ixz="-6.801394570971657e-18"/>
+    </inertial>
+    <!-- kept original visual transform to preserve cup frame convention -->
     <visual>
       <origin xyz="9.349037100037094e-10 0.004999995232077037 0.03650000482135752"
@@ -56,5 +65,5 @@
     <parent link="base_cad"/>
     <child link="arm_link"/>
-    <origin xyz="-0.3689156752862411 0.07293206200904699 -0.14265636918407304"
+    <origin xyz="-0.3689156752862411 0.07293206200904699 -0.14265636918407304" #maybe change vals (+20 and stuff)
             rpy="-1.5707963267948974 -1.5265566588595922e-16 7.21644966006352e-16"/>
     <axis xyz="0 0 1"/>
@@ -65,6 +74,10 @@
       <origin xyz="2.6474475234294913e-09 4.767925592119582e-09 -0.07580524145430977" rpy="0 0 0"/>
       <mass value="0.4797185340176825"/>
-      <inertia ixx="0.0011969873864993257" iyy="0.0009456324882451857" izz="0.0002533232197152197"
-               ixy="-1.3010426069826053e-18" iyz="1.734723475976807e-18" ixz="1.7802599672211983e-16"/>
+      <inertia ixx="0.0011969873864993257"
+               iyy="0.0009456324882451857"
+               izz="0.0002533232197152197"
+               ixy="-1.3010426069826053e-18"
+               iyz="1.734723475976807e-18"
+               ixz="1.7802599672211983e-16"/>
     </inertial>
     <visual>
@@ -172,10 +185,14 @@
       <origin xyz="-0.00013322161290098224 0.0009504573350092649 0.00043137020324471645" rpy="0 0 0"/>
       <mass value="0.0010174438167060709"/>
-      <inertia ixx="4.5307132551562007e-08" iyy="3.5090242032863035e-08" izz="7.59611441794051e-08"
-               ixy="1.0347644394329782e-09" iyz="-2.264070327162072e-09" ixz="1.3166586418150303e-10"/>
-    </inertial>
-    <visual>
-      <origin xyz="-2.352010142203653e-10 4.813011784676747e-09 -0.001750004628485895"
-              rpy="8.52607141014584e-18 -5.5511151231257815e-17 9.485990215114392e-16"/>
+      <inertia ixx="4.5307132551562007e-08"
+               iyy="3.5090242032863035e-08"
+               izz="7.59611441794051e-08"
+               ixy="1.0347644394329782e-09"
+               iyz="-2.264070327162072e-09"
+               ixz="1.3166586418150303e-10"/>
+    </inertial>
+    <visual>
+      <origin xyz="3.328162776483623e-09 -0.0026249951786425996 -0.0012500022897735264"
+              rpy="0 0 0"/>
       <geometry>
         <mesh filename="package://match/meshes/arducam_link-v3.stl" scale="0.001 0.001 0.001"/>
@@ -183,6 +200,6 @@
     </visual>
     <collision>
-      <origin xyz="-2.352010142203653e-10 4.813011784676747e-09 -0.001750004628485895"
-              rpy="8.52607141014584e-18 -5.5511151231257815e-17 9.485990215114392e-16"/>
+      <origin xyz="3.328162776483623e-09 -0.0026249951786425996 -0.0012500022897735264"
+              rpy="0 0 0"/>
       <geometry>
         <mesh filename="package://match/meshes/arducam_link-v3.stl" scale="0.001 0.001 0.001"/>
@@ -194,7 +211,7 @@
     <child link="arducam_link"/>
     <origin xyz="-0.2678761652862411 0.16593206200904703 0.06147094081592663"
-            rpy="-3.1415926535897922 -0.6973907898697068 -3.141592653589792"/>
-  </joint>
-  <!-- ROS optical frame for camera-based vision -->
+            rpy="-3.141592653589792 -0.7853981633974493 -3.141592653589792"/>
+  </joint>
+  <!-- ROS optical frame -->
   <link name="arducam_optical_frame"/>
   <joint name="arducam_to_optical" type="fixed">
@@ -255,20 +272,20 @@
     <parent link="arm_link"/>
     <child link="cup_0"/>
-    <origin xyz="0.075 0.0105 0.0365" rpy="1.5707963267948966 0 0"/>
+    <origin xyz="0.1 0.0255 0.0365" rpy="1.5707963267948966 0 0"/>
   </joint>
   <joint name="arm_to_cup_1" type="fixed">
     <parent link="arm_link"/>
     <child link="cup_1"/>
-    <origin xyz="0.025 0.0100 0.0365" rpy="-1.5707963267948966 0 0"/>
+    <origin xyz="0.05 0.025 0.0365" rpy="-1.5707963267948966 0 0"/>
   </joint>
   <joint name="arm_to_cup_2" type="fixed">
     <parent link="arm_link"/>
     <child link="cup_2"/>
-    <origin xyz="-0.025 0.0105 0.0365" rpy="1.5707963267948966 0 0"/>
+    <origin xyz="0 0.0255 0.0365" rpy="1.5707963267948966 0 0"/>
   </joint>
   <joint name="arm_to_cup_3" type="fixed">
     <parent link="arm_link"/>
     <child link="cup_3"/>
-    <origin xyz="-0.075 0.0105 0.0365" rpy="1.5707963267948966 0 0"/>
+    <origin xyz="-0.05 0.0255 0.0365" rpy="1.5707963267948966 0 0"/>
   </joint>
 </robot>

Commit message: cwa

File: server_ws/src/match/description/my_robot.urdf.xacro (robot description, xacro)
@@ -65,5 +65,5 @@
     <parent link="base_cad"/>
     <child link="arm_link"/>
-    <origin xyz="-0.3689156752862411 0.07293206200904699 -0.14265636918407304" #maybe change vals (+20 and stuff)
+    <origin xyz="-0.3689156752862411 0.07293206200904699 -0.14265636918407304" #maybe change vals (+20cm and stuff)
             rpy="-1.5707963267948974 -1.5265566588595922e-16 7.21644966006352e-16"/>
     <axis xyz="0 0 1"/>

Commit message: urdf cup alignment

File: server_ws/src/match/description/my_robot.urdf.xacro (robot description, xacro)
@@ -272,20 +272,20 @@
     <parent link="arm_link"/>
     <child link="cup_0"/>
-    <origin xyz="0.075 0.0255 0.0365" rpy="1.5707963267948966 0 0"/>
+    <origin xyz="0.075 0.0255 0.0027067937990953" rpy="1.5707963267948966 0 0"/>
   </joint>
   <joint name="arm_to_cup_1" type="fixed">
     <parent link="arm_link"/>
     <child link="cup_1"/>
-    <origin xyz="0.025 0.0255 0.0365" rpy="1.5707963267948966 0 0"/>
+    <origin xyz="0.025 0.0255 0.0027067937990953" rpy="1.5707963267948966 0 0"/>
   </joint>
   <joint name="arm_to_cup_2" type="fixed">
     <parent link="arm_link"/>
     <child link="cup_2"/>
-    <origin xyz="-0.025 0.0255 0.0365" rpy="1.5707963267948966 0 0"/>
+    <origin xyz="-0.025 0.0255 0.0027067937990953" rpy="1.5707963267948966 0 0"/>
   </joint>
   <joint name="arm_to_cup_3" type="fixed">
     <parent link="arm_link"/>
     <child link="cup_3"/>
-    <origin xyz="-0.075 0.0255 0.0365" rpy="1.5707963267948966 0 0"/>
+    <origin xyz="-0.075 0.0255 0.0027067937990953" rpy="1.5707963267948966 0 0"/>
   </joint>
 </robot>

Commit message: changes

File: server_ws/src/match/description/my_robot.urdf.xacro (robot description, xacro)
@@ -220,4 +220,11 @@
     <origin xyz="0 0 0" rpy="-1.57079632679 0 -1.57079632679"/>
   </joint>
+  <!-- ===================== LIDAR ===================== -->
+  <link name="laser_frame"/>
+  <joint name="base_to_laser" type="fixed">
+    <parent link="base_link"/>
+    <child link="laser_frame"/>
+    <origin xyz="-0.154078 -0.003064 0.0" rpy="0 0 0.0"/>
+  </joint>
   <!-- ===================== SUCTION CUPS ===================== -->
   <link name="cup_0">

Commit message: hardcoded tf

File: server_ws/src/match/description/my_robot.urdf.xacro (robot description, xacro)
@@ -220,11 +220,4 @@
     <origin xyz="0 0 0" rpy="-1.57079632679 0 -1.57079632679"/>
   </joint>
-  <!-- ===================== LIDAR ===================== -->
-  <link name="laser_frame"/>
-  <joint name="base_to_laser" type="fixed">
-    <parent link="base_link"/>
-    <child link="laser_frame"/>
-    <origin xyz="-0.154078 -0.003064 0.0" rpy="0 0 0.0"/>
-  </joint>
   <!-- ===================== SUCTION CUPS ===================== -->
   <link name="cup_0">
